Commit message: fixed urdf typo

File: gear_sonic/data/robot_model/model_data/g1/with_brainco/g1_29dof_with_hand.urdf (robot description, URDF)
Before this commit: robot g1_29dof_mode_15_brainco_hand, 73 links, 72 joints
Joints:
- removed joint right_thumb_tip
- added joint right_thumb_tip_joint: type revolute, parent right_thumb_distal_link, child right_thumb_tip, origin xyz=0 0.026529 -0.0017734 rpy=-0.06675 0 0, axis 1 0 0, limit lower=0 upper=0 effort=0 velocity=0

Commit message: wip

File: gear_sonic/data/robot_model/model_data/g1/with_brainco/g1_29dof_with_hand.urdf (robot description, URDF)
Before this commit: robot g1_29dof_mode_15_brainco_hand, 73 links, 72 joints
Joints:
- joint left_index_tip_joint: axis 0 1 0 -> (none); limit lower=1 upper=1 effort=1 velocity=1 -> (none); type revolute -> fixed
- joint left_middle_tip_joint: axis 0 1 0 -> (none); limit lower=1 upper=1 effort=1 velocity=1 -> (none); type revolute -> fixed
- joint left_pinky_tip_joint: axis 0 1 0 -> (none); limit lower=1 upper=1 effort=1 velocity=1 -> (none); type revolute -> fixed
- joint left_ring_tip_joint: axis 0 1 0 -> (none); limit lower=1 upper=1 effort=1 velocity=1 -> (none); type revolute -> fixed
- joint left_thumb_tip_joint: axis -1 0 0 -> (none); limit lower=0 upper=0 effort=0 velocity=0 -> (none); type revolute -> fixed
- joint right_index_tip_joint: axis 0 1 0 -> (none); limit lower=0 upper=0 effort=0 velocity=0 -> (none); type revolute -> fixed
- joint right_middle_tip_joint: axis 0 1 0 -> (none); limit lower=0 upper=0 effort=0 velocity=0 -> (none); type revolute -> fixed
- joint right_pinky_tip_joint: axis 0 1 0 -> (none); limit lower=0 upper=0 effort=0 velocity=0 -> (none); type revolute -> fixed
- joint right_ring_tip_joint: axis 0 1 0 -> (none); limit lower=0 upper=0 effort=0 velocity=0 -> (none); type revolute -> fixed
- joint right_thumb_tip_joint: axis 1 0 0 -> (none); limit lower=0 upper=0 effort=0 velocity=0 -> (none); type revolute -> fixed
